Commit message: camera adjustment

File: urdf/cluedo_robot.urdf (robot description, URDF)
Before this commit: robot cluedo_robot, 13 links, 12 joints
Joints:
- joint arm_joint_02: limit lower=-1.8 upper=1.8 effort=1000.0 velocity=0.2 -> lower=-2.8 upper=2.8 effort=1000.0 velocity=0.2
- joint arm_joint_03: limit lower=-1.8 upper=1.8 effort=1000.0 velocity=0.2 -> lower=-2.8 upper=2.8 effort=1000.0 velocity=0.2
- joint camera_joint2: origin xyz=0 0 0.05 rpy=0 0 0 -> xyz=0 0 0.05 rpy=0 0 1.57

File: urdf/cluedo_robot.xacro (robot description, xacro)
@@ -215,5 +215,5 @@
   <joint name="arm_joint_02" type="revolute">
   	<axis xyz="1 0 0"/>
-  	<limit effort="1000.0" lower="-1.8" upper="1.8" velocity="0.2"/>
+  	<limit effort="1000.0" lower="-2.8" upper="2.8" velocity="0.2"/>
   	<origin rpy="0 0 0" xyz="0 0 0.5"/>
   	<parent link="arm_link_01"/>
@@ -242,5 +242,5 @@
   <joint name="arm_joint_03" type="revolute">
   	<axis xyz="1 0 0"/>
-  	<limit effort="1000.0" lower="-1.8" upper="1.8" velocity="0.2"/>
+  	<limit effort="1000.0" lower="-2.8" upper="2.8" velocity="0.2"/>
   	<origin rpy="0 0 0" xyz="0 0 0.5"/>
   	<parent link="arm_link_02"/>
@@ -276,5 +276,5 @@
  <link name="camera_link2">
 	    <collision>
-	      <origin xyz="0 0 0.025" rpy="0 0 0"/>
+	      <origin xyz="0 0 0.025" rpy="0 0 -1.57"/>
 	      <geometry>
 		<box size="0.05 0.05 0.05"/>
@@ -282,5 +282,5 @@
 	    </collision>
 	    <visual>
-	      <origin xyz="0 0 0.025" rpy="0 0 0"/>
+	      <origin xyz="0 0 0.025" rpy="0 0 -1.57"/>
 	      <geometry>
 		<box size="0.05 0.05 0.05"/>
@@ -292,5 +292,5 @@
 	    <inertial>
 	      <mass value="1e-5" />
-	      <origin xyz="0 0 0" rpy="0 0 0"/>
+	      <origin xyz="0 0 0" rpy="0 0 -1.57"/>
 	      <inertia ixx="1e-6" ixy="0" ixz="0" iyy="1e-6" iyz="0" izz="1e-6" />
 	    </inertial>
@@ -298,5 +298,5 @@
   <joint name="camera_joint2" type="fixed">
 	    <axis xyz="0 1 0" />
-	    <origin xyz="0 0 0.05" rpy="0 0 0"/>
+	    <origin xyz="0 0 0.05" rpy="0 0 1.57"/>
 	    <parent link="cluedo_link"/>
 	    <child link="camera_link2"/>
